File: hardware/v0.1/bb_v0.1.kicad_pcb (KiCad board)
At the start: 2 copper layers, 65 x 45 mm, 57 parts, among them J1 USB_B_Micro, Q1 MMBT4403_, SW1 SW_Omron_B3FS, U1 MCP1640Cx-xCHY, U2 MAX16054AZT_T, U3 ESP32-C3-WROOM-02, U4 HX711

Commit message: added button
Parts:
- added C15: 100n, Capacitor_SMD:C_0603_1608Metric_Pad1.08x0.95mm_HandSolder, F.Cu at (67.0, 90.4)
- added SW2: SW_Omron_B3FS, Button_Switch_SMD:SW_SPST_Omron_B3FS-101xP, F.Cu at (61.0, 90.0)
- moved D4 64.7 mm to (111.5, 60.1)
- moved R7 61.1 mm to (113.5, 60.1), turned to 90 degrees
- moved D5 60.4 mm to (109.5, 60.1)
- moved R8 54.1 mm to (107.5, 60.1), turned to 90 degrees
- moved C6 16.8 mm to (79.0, 78.4), turned to -90 degrees
- moved C7 14.7 mm to (80.5, 78.4), turned to -90 degrees
- moved R3 12.8 mm to (82.0, 78.4), turned to 90 degrees
- moved C5 10.8 mm to (83.5, 78.4), turned to -90 degrees
- moved C4 1.00 mm to (70.0, 59.5)
- moved C3 0.50 mm to (65.0, 59.5)
Routing:
- net /GPIO4: track 12.9 -> 52.5 mm
- net /GPIO9: track 0.00 -> 39.4 mm, vias 0 -> 3
- net Net-(U3-EN): track 0.00 -> 23.4 mm, vias 0 -> 2
- net /GPIO8: track 0.00 -> 9.66 mm, vias 0 -> 2
- net /AVDD: track 25.8 -> 29.7 mm
- net Net-(D4-A): track 4.88 -> 2.02 mm
- net Net-(D5-A): track 3.88 -> 2.02 mm
- net /3V3: track 129.7 -> 128.7 mm, vias 2 -> 4
- net /D-: track 10.7 -> 9.74 mm
- net /D+: track 10.1 -> 9.60 mm
Other:
- board text added: "- A+"
- board text added: "- A-"
- board text added: "- B+"
- board text added: "- B-"
- board text added: "- E+"
- board text added: "- E-"
- board text added: "- SHIELD"
- board text added: "BigBanger v0.1"

Commit message: first version complete layout
Parts:
- moved D4 4.50 mm to (107.0, 60.1)
- moved D5 4.50 mm to (105.0, 60.1)
- moved R7 4.50 mm to (109.0, 60.1)
- moved R8 4.50 mm to (103.0, 60.1)
Routing:
- net GND: track 4.10 -> 65.4 mm, vias 0 -> 81
- net /GPIO4: track 52.5 -> 49.7 mm
- net /3V3: track 128.7 -> 129.8 mm
- added copper zone on B.Cu, net GND
- added copper zone on F.Cu, net GND
Other:
- board text added: "github.com/FilMarini/bigbanger"
