File: hardware/v0.1/bb_v0.1.kicad_pcb (KiCad board)
At the start: 2 copper layers, 65 x 45 mm, 59 parts, among them J1 USB_B_Micro, Q1 MMBT4403_, SW1 SW_Omron_B3FS, SW2 SW_Omron_B3FS, U1 MCP1640Cx-xCHY, U2 MAX16054AZT_T, U3 ESP32-C3-WROOM-02, U4 HX711

Commit message: fixed oversights after first iteration
Parts:
- removed R4, R5: 0, Resistor_SMD:R_0603_1608Metric_Pad0.98x0.95mm_HandSolder
- U1: value MCP1640Cx-xCHY -> MCP1640Bx-xCHY
- moved J1 46.8 mm to (112.0, 63.5), turned to 90 degrees
- moved D1 43.1 mm to (108.0, 61.4), turned to 90 degrees
- moved C3 41.5 mm to (106.5, 61.0), turned to 90 degrees
- moved D2 39.9 mm to (108.0, 65.7), turned to -90 degrees
- moved C4 37.1 mm to (106.5, 66.0), turned to -90 degrees
- moved TP3 19.2 mm to (63.5, 55.0)
- moved TP4 19.2 mm to (66.5, 55.0)
- moved TP7 16.9 mm to (60.0, 52.5)
- moved TP1 16.4 mm to (57.0, 52.5)
- moved TP5 16.3 mm to (72.5, 55.0)
- moved TP2 10.4 mm to (69.5, 55.0)
- moved TP6 8.14 mm to (97.0, 52.0)
- moved D3 4.53 mm to (98.5, 60.6)
- moved D4 4.53 mm to (100.5, 60.6)
- moved D5 4.53 mm to (102.5, 60.6)
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Connections:
- SW1 pad 1: /BATT3V -> GND
- U3 pad 11: Net-(U3-IO20/RXD) -> unconnected-(U3-IO20/RXD-Pad11)
- U3 pad 12: Net-(U3-IO21/TXD) -> unconnected-(U3-IO21/TXD-Pad12)
Routing:
- net /D+: track 9.60 -> 55.7 mm
- net /D-: track 9.74 -> 53.7 mm
- net /AVDD: track 29.7 -> 49.4 mm
- net /A-: track 8.11 -> 23.0 mm
- net /A+: track 8.61 -> 21.3 mm
- net Net-(U3-IO21/TXD): track 9.03 -> 0.00 mm
- net Net-(U3-IO20/RXD): track 4.95 -> 0.00 mm
- net /GPIO4: track 50.5 -> 47.0 mm
- net /BATT3V: track 105.0 -> 106.1 mm
- net /3V3: track 135.1 -> 134.1 mm
- net /A3V3EN: track 7.23 -> 6.38 mm
- net GND: track 80.2 -> 81.0 mm, vias 85 -> 82
- net /SWOUT: track 33.9 -> 33.3 mm
Other:
- outline, holes or cut-outs redrawn
- board text added: "B+"
- board text added: "B-"
- board text removed: "- B+"
- board text removed: "- B-"

Commit message: v1.0
Parts:
- moved H2 0.50 mm to (52.5, 86.0)
- moved H5 0.50 mm to (98.0, 86.0)
Routing:
- net GND: track 81.0 -> 87.2 mm, vias 82 -> 85
Changed lines of the file:
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@@
 	(footprint "MountingHole:MountingHole_2.2mm_M2"
 		(layer "F.Cu")
-		(at 52.5 86.5)
+		(at 52.5 86)
 		(descr "Mounting Hole 2.2mm, no annular, M2")
 		(tags "mounting hole 2.2mm no annular m2")
@@
 	(footprint "MountingHole:MountingHole_2.2mm_M2"
 		(layer "F.Cu")
-		(at 98 86.5)
+		(at 98 86)
 		(descr "Mounting Hole 2.2mm, no annular, M2")
 		(tags "mounting hole 2.2mm no annular m2")
@@
 	)
 	(segment
+		(start 110.6 60.1)
+		(end 110 59.5)
+		(width 0.18)
+		(layer "F.Cu")
+		(net 1)
+	)
+	(segment
 		(start 80.5 77.5)
 		(end 80.456344 77.5)
@@
 	)
 	(segment
-		(start 114.41 66.86)
-		(end 114.41 67.59)
-		(width 0.18)
-		(layer "F.Cu")
-		(net 1)
-	)
-	(segment
 		(start 56.5 90.1375)
 		(end 56.5 89.5)
@@
 	)
 	(segment
-		(start 110.6 62.2)
-		(end 113 62.2)
+		(start 110.6 61)
+		(end 110.6 60.1)
 		(width 0.18)
 		(layer "F.Cu")
@@
 	)
 	(segment
-		(start 114.075 66.525)
-		(end 114.41 66.86)
+		(start 110.6 62.2)
+		(end 113 62.2)
 		(width 0.18)
 		(layer "F.Cu")
@@
 	)
 	(segment
+		(start 113.3 67)
+		(end 113.3 67.7)
+		(width 0.18)
+		(layer "F.Cu")
+		(net 1)
+	)
+	(segment
 		(start 100.5 67.66)
 		(end 101.544473 68.704473)
@@
 	)
 	(segment
+		(start 113.3 67.7)
+		(end 112.5 68.5)
+		(width 0.18)
+		(layer "F.Cu")
+		(net 1)
+	)
+	(segment
 		(start 101.45 68.2)
 		(end 102.25 69)
@@
 	)
 	(segment
+		(start 110.6 67.9)
+		(end 110.5 68)
+		(width 0.18)
+		(layer "F.Cu")
+		(net 1)
+	)
+	(segment
+		(start 110.6 66)
+		(end 110.6 67.9)
+		(width 0.18)
+		(layer "F.Cu")
+		(net 1)
+	)
+	(segment
 		(start 100.5 61.73)
 		(end 101 62.23)
@@
 	)
 	(segment
-		(start 114.41 67.59)
-		(end 114 68)
-		(width 0.18)
-		(layer "F.Cu")
-		(net 1)
-	)
-	(segment
 		(start 109 75.32)
 		(end 108.82 75.5)
@@
 	)
 	(segment
+		(start 113.3 58.8)
+		(end 112.5 58)
+		(width 0.18)
+		(layer "F.Cu")
+		(net 1)
+	)
+	(segment
+		(start 113.3 60)
+		(end 113.3 58.8)
+		(width 0.18)
+		(layer "F.Cu")
+		(net 1)
+	)
+	(segment
 		(start 101.544473 68.704473)
 		(end 101.544473 69.455527)
@@
 	)
 	(via
+		(at 110.5 68)
+		(size 0.8)
+		(drill 0.3)
+		(layers "F.Cu" "B.Cu")
+		(net 1)
+	)
+	(via
 		(at 87.5 80)
 		(size 0.8)
@@
 	)
 	(via
-		(at 114 68)
+		(at 112.5 68.5)
 		(size 0.8)
 		(drill 0.3)
 		(layers "F.Cu" "B.Cu")
-		(free yes)
 		(net 1)
 	)
@@
 	)
 	(via
+		(at 110 59.5)
+		(size 0.8)
+		(drill 0.3)
+		(layers "F.Cu" "B.Cu")
+		(net 1)
+	)
+	(via
 		(at 84.5 77.5)
 		(size 0.8)
@@
 	)
 	(via
+		(at 112.5 58)
+		(size 0.8)
+		(drill 0.3)
+		(layers "F.Cu" "B.Cu")
+		(net 1)
+	)
+	(via
 		(at 76.5 61)
 		(size 0.8)
@@
 	)
 	(via
-		(at 112 57)
+		(at 110 56)
 		(size 0.8)
 		(drill 0.3)
