File: hardware/v0.1/WeilHeng_WH-C07/bb_v0.1.kicad_pcb (KiCad board)
At the start: 2 copper layers, 65 x 45 mm, 59 parts, among them J1 USB_B_Micro, Q1 MMBT4403_, SW1 SW_Omron_B3FS, SW2 SW_Omron_B3FS, U1 MCP1640Cx-xCHY, U2 MAX16054AZT_T, U3 ESP32-C3-WROOM-02, U4 HX711

Commit message: checked measures
Parts:
- moved C15 10.5 mm to (56.5, 91.0)
- moved R7 10.0 mm to (99.0, 60.2)
- moved D3 7.27 mm to (103.0, 60.1)
- moved R6 6.78 mm to (97.0, 60.2), turned to 90 degrees
- moved R8 2.00 mm to (101.0, 60.2)
- moved D4 2.00 mm to (105.0, 60.1)
- moved D5 2.00 mm to (107.0, 60.1)
- moved SW2 2.00 mm to (63.0, 90.0)
- moved R4 1.00 mm to (78.0, 60.0)
- moved R5 1.00 mm to (76.0, 60.0)
- moved SW1 1.00 mm to (105.0, 90.0)
- moved H1 0.71 mm to (112.0, 87.5)
- moved H3 0.71 mm to (52.5, 52.5)
- moved H5 0.71 mm to (98.0, 87.5)
- moved H2 0.50 mm to (52.5, 87.5)
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Routing:
- net Net-(D3-A): track 4.20 -> 19.9 mm
- net GND: track 65.4 -> 80.2 mm, vias 81 -> 85
- net Net-(D5-A): track 2.02 -> 8.34 mm
- net /BATT3V: track 110.5 -> 105.0 mm
- net /3V3: track 129.8 -> 135.1 mm
- net Net-(D4-A): track 2.02 -> 6.67 mm
- net /A3V3EN: track 11.6 -> 7.23 mm
- net /GPIO9: track 39.4 -> 41.8 mm
- net /GPIO4: track 49.7 -> 50.5 mm
