File: hardware/bb_kicad/bb_kicad.kicad_pcb (KiCad board)
At the start: 2 copper layers, 65 x 45 mm, 57 parts, among them J1 USB_B_Micro, Q1 MMBT4403_, SW1 SW_Omron_B3FS, SW2 SW_Omron_B3FS, U1 MCP1640Bx-xCHY, U2 MAX16054AZT_T, U3 ESP32-C3-WROOM-02, U4 HX711

Commit message: changed project name and version
Other:
- board text added: "BigBanger v1.0"
- board text removed: "BigBanger v0.1"
Changed lines of the file:
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@@
 		)
 	)
-	(gr_text "BigBanger\nv0.1"
+	(gr_text "BigBanger\nv1.0"
 		(at 74.5 76.5 0)
 		(layer "F.SilkS")
